Commit message: Changed package name

File: description/urdf/gundam.urdf (robot description, URDF)
Before this commit: robot GGC_TestModel_rx78_20170112, 98 links, 97 joints
Links:
- link rx78_Null_001_link: geometry collision mesh filename=package://gundam_rx78_description/meshes/rx78_object_001-li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; visual mesh filename=package://gundam_rx78_description/meshes/rx78_object_001-li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
- link rx78_Null_002_link: geometry collision mesh filename=package://gundam_rx78_description/meshes/rx78_object_002-li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; visual mesh filename=package://gundam_rx78_description/meshes/rx78_object_002-li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
- link rx78_Null_003_link: geometry collision mesh filename=package://gundam_rx78_description/meshes/rx78_object_062-li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; visual mesh filename=package://gundam_rx78_description/meshes/rx78_object_062-li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
- link rx78_Null_004_link: geometry collision mesh filename=package://gundam_rx78_description/meshes/rx78_object_063-li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; visual mesh filename=package://gundam_rx78_description/meshes/rx78_object_063-li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
- link rx78_Null_005_link: geometry collision mesh filename=package://gundam_rx78_description/meshes/rx78_object_005-li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; visual mesh filename=package://gundam_rx78_description/meshes/rx78_object_005-li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
- link rx78_Null_006_link: geometry collision mesh filename=package://gundam_rx78_description/meshes/rx78_object_004-li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; visual mesh filename=package://gundam_rx78_description/meshes/rx78_object_004-li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
- link rx78_Null_008_link: geometry collision mesh filename=package://gundam_rx78_description/meshes/rx78_object_006-li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; visual mesh filename=package://gundam_rx78_description/meshes/rx78_object_006-li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
- link rx78_Null_010_link: geometry collision mesh filename=package://gundam_rx78_description/meshes/rx78_object_007-li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; visual mesh filename=package://gundam_rx78_description/meshes/rx78_object_007-li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
- link rx78_Null_013_link: geometry collision mesh filename=package://gundam_rx78_description/meshes/rx78_object_003-li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; visual mesh filename=package://gundam_rx78_description/meshes/rx78_object_003-li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
- link rx78_Null_014_link: geometry collision mesh filename=package://gundam_rx78_description/meshes/rx78_object_011-li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; visual mesh filename=package://gundam_rx78_description/meshes/rx78_object_011-li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
- link rx78_Null_015_link: geometry collision mesh filename=package://gundam_rx78_description/meshes/rx78_object_008-li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; visual mesh filename=package://gundam_rx78_description/meshes/rx78_object_008-li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
- link rx78_Null_016_link: geometry collision mesh filename=package://gundam_rx78_description/meshes/rx78_object_080-li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; visual mesh filename=package://gundam_rx78_description/meshes/rx78_object_080-li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
- link rx78_Null_017_link: geometry collision mesh filename=package://gundam_rx78_description/meshes/rx78_object_083-li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; visual mesh filename=package://gundam_rx78_description/meshes/rx78_object_083-li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
- link rx78_Null_018_link: geometry collision mesh filename=package://gundam_rx78_description/meshes/rx78_object_084-li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; visual mesh filename=package://gundam_rx78_description/meshes/rx78_object_084-li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
- link rx78_Null_021_link: geometry collision mesh filename=package://gundam_rx78_description/meshes/rx78_object_014-li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; visual mesh filename=package://gundam_rx78_description/meshes/rx78_object_014-li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
- link rx78_Null_022_link: geometry collision mesh filename=package://gundam_rx78_description/meshes/rx78_object_013-li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; visual mesh filename=package://gundam_rx78_description/meshes/rx78_object_013-li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
- link rx78_Null_023_link: geometry collision mesh filename=package://gundam_rx78_description/meshes/rx78_object_012-li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; visual mesh filename=package://gundam_rx78_description/meshes/rx78_object_012-li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
- link rx78_Null_024_link: geometry collision mesh filename=package://gundam_rx78_description/meshes/rx78_object_017-li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; visual mesh filename=package://gundam_rx78_description/meshes/rx78_object_017-li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
- link rx78_Null_025_link: geometry collision mesh filename=package://gundam_rx78_description/meshes/rx78_object_016-li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; visual mesh filename=package://gundam_rx78_description/meshes/rx78_object_016-li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
- link rx78_Null_026_link: geometry collision mesh filename=package://gundam_rx78_description/meshes/rx78_object_015-li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; visual mesh filename=package://gundam_rx78_description/meshes/rx78_object_015-li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
- link rx78_Null_027_link: geometry collision mesh filename=package://gundam_rx78_description/meshes/rx78_object_020-li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; visual mesh filename=package://gundam_rx78_description/meshes/rx78_object_020-li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
- link rx78_Null_028_link: geometry collision mesh filename=package://gundam_rx78_description/meshes/rx78_object_019-li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; visual mesh filename=package://gundam_rx78_description/meshes/rx78_object_019-li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
- link rx78_Null_029_link: geometry collision mesh filename=package://gundam_rx78_description/meshes/rx78_object_018-li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; visual mesh filename=package://gundam_rx78_description/meshes/rx78_object_018-li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
- link rx78_Null_030_link: geometry collision mesh filename=package://gundam_rx78_description/meshes/rx78_object_021-li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; visual mesh filename=package://gundam_rx78_description/meshes/rx78_object_021-li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
- link rx78_Null_031_link: geometry collision mesh filename=package://gundam_rx78_description/meshes/rx78_object_025-li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; visual mesh filename=package://gundam_rx78_description/meshes/rx78_object_025-li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
- link rx78_Null_032_link: geometry collision mesh filename=package://gundam_rx78_description/meshes/rx78_object_026-li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; visual mesh filename=package://gundam_rx78_description/meshes/rx78_object_026-li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
- link rx78_Null_033_link: geometry collision mesh filename=package://gundam_rx78_description/meshes/rx78_object_027-li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; visual mesh filename=package://gundam_rx78_description/meshes/rx78_object_027-li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
- link rx78_Null_034_link: geometry collision mesh filename=package://gundam_rx78_description/meshes/rx78_object_028-li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; visual mesh filename=package://gundam_rx78_description/meshes/rx78_object_028-li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
- link rx78_Null_035_link: geometry collision mesh filename=package://gundam_rx78_description/meshes/rx78_object_029-li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; visual mesh filename=package://gundam_rx78_description/meshes/rx78_object_029-li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
- link rx78_Null_036_link: geometry collision mesh filename=package://gundam_rx78_description/meshes/rx78_object_042-li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; visual mesh filename=package://gundam_rx78_description/meshes/rx78_object_042-li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
- link rx78_Null_037_link: geometry collision mesh filename=package://gundam_rx78_description/meshes/rx78_object_041-li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; visual mesh filename=package://gundam_rx78_description/meshes/rx78_object_041-li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
- link rx78_Null_038_link: geometry collision mesh filename=package://gundam_rx78_description/meshes/rx78_object_030-li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; visual mesh filename=package://gundam_rx78_description/meshes/rx78_object_030-li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
- link rx78_Null_039_link: geometry collision mesh filename=package://gundam_rx78_description/meshes/rx78_object_040-li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; visual mesh filename=package://gundam_rx78_description/meshes/rx78_object_040-li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
- link rx78_Null_040_link: geometry collision mesh filename=package://gundam_rx78_description/meshes/rx78_object_032-li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; visual mesh filename=package://gundam_rx78_description/meshes/rx78_object_032-li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
- link rx78_Null_041_link: geometry collision mesh filename=package://gundam_rx78_description/meshes/rx78_object_034-li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; visual mesh filename=package://gundam_rx78_description/meshes/rx78_object_034-li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
- link rx78_Null_046_link: geometry collision mesh filename=package://gundam_rx78_description/meshes/rx78_object_039-li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; visual mesh filename=package://gundam_rx78_description/meshes/rx78_object_039-li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
- link rx78_Null_047_link: geometry collision mesh filename=package://gundam_rx78_description/meshes/rx78_object_043-li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; visual mesh filename=package://gundam_rx78_description/meshes/rx78_object_043-li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
- link rx78_Null_048_link: geometry collision mesh filename=package://gundam_rx78_description/meshes/rx78_object_045-li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; visual mesh filename=package://gundam_rx78_description/meshes/rx78_object_045-li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
- link rx78_Null_049_link: geometry collision mesh filename=package://gundam_rx78_description/meshes/rx78_object_078-li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; visual mesh filename=package://gundam_rx78_description/meshes/rx78_object_078-li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
- link rx78_Null_050_link: geometry collision mesh filename=package://gundam_rx78_description/meshes/rx78_object_046-li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; visual mesh filename=package://gundam_rx78_description/meshes/rx78_object_046-li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
- link rx78_Null_051_link: geometry collision mesh filename=package://gundam_rx78_description/meshes/rx78_object_077-li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; visual mesh filename=package://gundam_rx78_description/meshes/rx78_object_077-li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
- link rx78_Null_052_link: geometry collision mesh filename=package://gundam_rx78_description/meshes/rx78_object_076-li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; visual mesh filename=package://gundam_rx78_description/meshes/rx78_object_076-li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
- link rx78_Null_053_link: geometry collision mesh filename=package://gundam_rx78_description/meshes/rx78_object_075-li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; visual mesh filename=package://gundam_rx78_description/meshes/rx78_object_075-li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
- link rx78_Null_054_link: geometry collision mesh filename=package://gundam_rx78_description/meshes/rx78_object_047-li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; visual mesh filename=package://gundam_rx78_description/meshes/rx78_object_047-li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
- link rx78_Null_055_link: geometry collision mesh filename=package://gundam_rx78_description/meshes/rx78_object_048-li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; visual mesh filename=package://gundam_rx78_description/meshes/rx78_object_048-li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
- link rx78_Null_056_link: geometry collision mesh filename=package://gundam_rx78_description/meshes/rx78_object_051-li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; visual mesh filename=package://gundam_rx78_description/meshes/rx78_object_051-li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
- link rx78_Null_057_link: geometry collision mesh filename=package://gundam_rx78_description/meshes/rx78_object_050-li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; visual mesh filename=package://gundam_rx78_description/meshes/rx78_object_050-li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
- link rx78_Null_058_link: geometry collision mesh filename=package://gundam_rx78_description/meshes/rx78_object_049-li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; visual mesh filename=package://gundam_rx78_description/meshes/rx78_object_049-li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
- link rx78_Null_059_link: geometry collision mesh filename=package://gundam_rx78_description/meshes/rx78_object_056-li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; visual mesh filename=package://gundam_rx78_description/meshes/rx78_object_056-li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
- link rx78_Null_060_link: geometry collision mesh filename=package://gundam_rx78_description/meshes/rx78_object_055-li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; visual mesh filename=package://gundam_rx78_description/meshes/rx78_object_055-li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
- link rx78_Null_061_link: geometry collision mesh filename=package://gundam_rx78_description/meshes/rx78_object_054-li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; visual mesh filename=package://gundam_rx78_description/meshes/rx78_object_054-li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
- link rx78_Null_062_link: geometry collision mesh filename=package://gundam_rx78_description/meshes/rx78_object_059-li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; visual mesh filename=package://gundam_rx78_description/meshes/rx78_object_059-li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
- link rx78_Null_063_link: geometry collision mesh filename=package://gundam_rx78_description/meshes/rx78_object_058-li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; visual mesh filename=package://gundam_rx78_description/meshes/rx78_object_058-li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
- link rx78_Null_064_link: geometry collision mesh filename=package://gundam_rx78_description/meshes/rx78_object_057-li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; visual mesh filename=package://gundam_rx78_description/meshes/rx78_object_057-li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
- link rx78_Null_066_link: geometry collision mesh filename=package://gundam_rx78_description/meshes/rx78_object_064-li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; visual mesh filename=package://gundam_rx78_description/meshes/rx78_object_064-li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
- link rx78_Null_067_link: geometry collision mesh filename=package://gundam_rx78_description/meshes/rx78_object_061-li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; visual mesh filename=package://gundam_rx78_description/meshes/rx78_object_061-li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
- link rx78_Null_068_link: geometry collision mesh filename=package://gundam_rx78_description/meshes/rx78_object_067-li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; visual mesh filename=package://gundam_rx78_description/meshes/rx78_object_067-li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
- link rx78_Null_069_link: geometry collision mesh filename=package://gundam_rx78_description/meshes/rx78_object_060-li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; visual mesh filename=package://gundam_rx78_description/meshes/rx78_object_060-li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
- link rx78_Null_070_link: geometry collision mesh filename=package://gundam_rx78_description/meshes/rx78_object_066-li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; visual mesh filename=package://gundam_rx78_description/meshes/rx78_object_066-li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
- link rx78_Null_071_link: geometry collision mesh filename=package://gundam_rx78_description/meshes/rx78_object_065-li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; visual mesh filename=package://gundam_rx78_description/meshes/rx78_object_065-li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
- link rx78_Null_072_link: geometry collision mesh filename=package://gundam_rx78_description/meshes/rx78_object_070-li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; visual mesh filename=package://gundam_rx78_description/meshes/rx78_object_070-li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
- link rx78_Null_073_link: geometry collision mesh filename=package://gundam_rx78_description/meshes/rx78_object_069-li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; visual mesh filename=package://gundam_rx78_description/meshes/rx78_object_069-li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
- link rx78_Null_074_link: geometry collision mesh filename=package://gundam_rx78_description/meshes/rx78_object_068-li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; visual mesh filename=package://gundam_rx78_description/meshes/rx78_object_068-li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
- link rx78_Null_075_link: geometry collision mesh filename=package://gundam_rx78_description/meshes/rx78_object_053-li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; visual mesh filename=package://gundam_rx78_description/meshes/rx78_object_053-li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
- link rx78_Null_076_link: geometry collision mesh filename=package://gundam_rx78_description/meshes/rx78_object_052-li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; visual mesh filename=package://gundam_rx78_description/meshes/rx78_object_052-li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
- link rx78_Null_077_link: geometry collision mesh filename=package://gundam_rx78_description/meshes/rx78_object_071-li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; visual mesh filename=package://gundam_rx78_description/meshes/rx78_object_071-li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
- link rx78_Null_078_link: geometry collision mesh filename=package://gundam_rx78_description/meshes/rx78_object_074-li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; visual mesh filename=package://gundam_rx78_description/meshes/rx78_object_074-li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
- link rx78_Null_079_link: geometry collision mesh filename=package://gundam_rx78_description/meshes/rx78_object_073-li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; visual mesh filename=package://gundam_rx78_description/meshes/rx78_object_073-li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
- link rx78_Null_080_link: geometry collision mesh filename=package://gundam_rx78_description/meshes/rx78_object_072-li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; visual mesh filename=package://gundam_rx78_description/meshes/rx78_object_072-li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
- link rx78_Null_081_link: geometry collision mesh filename=package://gundam_rx78_description/meshes/rx78_object_079-li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; visual mesh filename=package://gundam_rx78_description/meshes/rx78_object_079-li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
- link rx78_Null_083_link: geometry collision mesh filename=package://gundam_rx78_description/meshes/rx78_object_044-li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; visual mesh filename=package://gundam_rx78_description/meshes/rx78_object_044-li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
- link rx78_Null_084_link: geometry collision mesh filename=package://gundam_rx78_description/meshes/rx78_object_085-li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; visual mesh filename=package://gundam_rx78_description/meshes/rx78_object_085-li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
- link rx78_Null_085_link: geometry collision mesh filename=package://gundam_rx78_description/meshes/rx78_object_086-li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; visual mesh filename=package://gundam_rx78_description/meshes/rx78_object_086-li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
- link rx78_Null_086_link: geometry collision mesh filename=package://gundam_rx78_description/meshes/rx78_object_024-li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; visual mesh filename=package://gundam_rx78_description/meshes/rx78_object_024-li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
- link rx78_Null_087_link: geometry collision mesh filename=package://gundam_rx78_description/meshes/rx78_object_023-li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; visual mesh filename=package://gundam_rx78_description/meshes/rx78_object_023-li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
- link rx78_Null_088_link: geometry collision mesh filename=package://gundam_rx78_description/meshes/rx78_object_087-li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; visual mesh filename=package://gundam_rx78_description/meshes/rx78_object_087-li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
- link rx78_Null_089_link: geometry collision mesh filename=package://gundam_rx78_description/meshes/rx78_object_022-li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; visual mesh filename=package://gundam_rx78_description/meshes/rx78_object_022-li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
- link rx78_Null_090_link: geometry collision mesh filename=package://gundam_rx78_description/meshes/rx78_object_089-li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; visual mesh filename=package://gundam_rx78_description/meshes/rx78_object_089-li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
- link rx78_Null_091_link: geometry collision mesh filename=package://gundam_rx78_description/meshes/rx78_object_091-li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; visual mesh filename=package://gundam_rx78_description/meshes/rx78_object_091-li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
